File: hardware/keyboard_right/ergoducks_keyboard_right.kicad_sch (KiCad schematic)
At the start: 24 parts, among them J101 Conn_01x02, U102 SN74LV1T125DCKR

Commit message: Update after producion of rev 2
Parts:
- removed C101, C102, C103, C106, C107, C108: 100nF, Capacitor_SMD:C_0603_1608Metric_Pad1.08x0.95mm_HandSolder, symbol Device:C_Small
- removed EXTRA102: Conn_01x05, Connector_PinHeader_2.54mm:PinHeader_1x05_P2.54mm_Vertical, symbol Connector_Generic:Conn_01x05
- removed H105, H106: MountingHole, prettylib:mounting_hole, symbol Mechanical:MountingHole
- removed LINK101: SW_Push, prettylib:SW_SPST_CK_RS282G05A3_reversible, symbol Switch:SW_Push
- removed SYSOFF101: SW_SPST, Button_Switch_SMD:SW_DIP_SPSTx01_Slide_6.7x4.1mm_W6.73mm_P2.54mm_LowProfile_JPin, symbol Switch:SW_SPST
- added FID101, FID102, FID103: Fiducial, Fiducial:Fiducial_0.5mm_Mask1mm, symbol Mechanical:Fiducial
- added R101, R102: 1k, Resistor_SMD:R_0603_1608Metric_Pad0.98x0.95mm_HandSolder, symbol Device:R
- added SW101: RotaryEncoder, Rotary_Encoder:RotaryEncoder_Alps_EC11E-Switch_Vertical_H20mm_MountingHoles, symbol Device:RotaryEncoder
- added SWSYSOFF101: SW_SPDT, Button_Switch_SMD:SW_SPDT_CK_JS102011SAQN, symbol Switch:SW_SPDT
- C104: renamed from C105; footprint Capacitor_SMD:C_0603_1608Metric_Pad1.08x0.95mm_HandSolder -> Capacitor_SMD:C_0402_1005Metric; LCSC (none) -> C1525
- C105: renamed from C104; footprint Capacitor_SMD:C_0603_1608Metric_Pad1.08x0.95mm_HandSolder -> Capacitor_SMD:C_0402_1005Metric; LCSC (none) -> C1525
- H101, H102, H103, H104: footprint prettylib:mounting_hole -> MountingHole:MountingHole_2.2mm_M2
- J101, OLED101: now not fitted
- R103: renamed from R101; LCSC (none) -> C23025
- RESET101: footprint prettylib:SW_SPST_CK_RS282G05A3_reversible -> Button_Switch_SMD:SW_SPST_B3U-1000P-B; Digikey partno CKN10384CT-ND -> (none); LCSC (none) -> C561515; MANUFACTURER C&K -> XKB; Mouser partno 611-RS-282G05A3-SMRT -> (none); Product name RS-282G05A3-SM RT -> TS-3025-A-A-A
- U102: LCSC (none) -> C75925
Connections:
- net BUTTON is gone; now on net ROW3: U101.8 (P109)
- net +3V3: now also R101.2, R102.2
- net BACKLIGHT_DATA: now also U101.3 (P026); no longer U101.2 (P004)
- net EXT_INT: no longer U101.3 (P026)
- net GND: now also SW101.C, SWSYSOFF101.3 (C)
- net ROW0: now also U101.2 (P004); no longer U101.9 (P012)
- net ROW1: now also U101.6 (P006); no longer U101.10 (P013)
- net ROW2: now also U101.7 (P008); no longer U101.11 (P015)
- net ROW3: no longer U101.12 (P020)
- net ROW4: now also U101.9 (P012); no longer U101.13 (P017)
- net SYSOFF: now also SWSYSOFF101.2 (B)
- net TWI_SCL: now also U101.11 (P015); no longer U101.7 (P008)
- net TWI_SDA: now also U101.10 (P013); no longer U101.6 (P006)
- net VBAT+: now reaches J101.1 (Pin_1), U101.14 (BAT+)
- net COL7: now reaches U101.26 (P112)
- new net ENCA: R102.1, SW101.A, U101.12 (P020)
- new net ENCB: R101.1, SW101.B, U101.13 (P017)
- no-connect marks 0 -> 1
Other:
- added sheet switch36 (switch_1u.kicad_sch)
- added sheet switch37 (switch_1u.kicad_sch)
- added sheet switch38 (switch_1u.kicad_sch)
- added sheet switch39 (switch_1u.kicad_sch)
- added sheet switch40 (switch_1.5u.kicad_sch)
- sheet switch1: file switch_1.5u.kicad_sch -> switch_1u.kicad_sch
- sheet switch15: file switch_1.5u.kicad_sch -> switch_1u.kicad_sch
- sheet switch22: file switch_1.5u.kicad_sch -> switch_1u.kicad_sch
- sheet switch29: file switch_1.5u.kicad_sch -> switch_1u.kicad_sch
- sheet switch34: file switch_1.5u.kicad_sch -> switch_1u.kicad_sch
- sheet switch8: file switch_1.5u.kicad_sch -> switch_1u.kicad_sch
- moved on the sheet: C104, R103, U101, U102
